Commit message: Fixed robot description, converted meshes to supported format

File: irp6_description/robots/irp6pboth.urdf.xacro (robot description, xacro)
@@ -1,23 +1,6 @@
 <?xml version="1.0"?>
-<robot name="irp6"
-       xmlns:sensor="http://playerstage.sourceforge.net/gazebo/xmlschema/#sensor"
-       xmlns:controller="http://playerstage.sourceforge.net/gazebo/xmlschema/#controller"
-       xmlns:xacro="http://ros.org/wiki/fixme"
-       xmlns:interface="http://playerstage.sourceforge.net/gazebo/xmlschema/#interface">
+<robot name="irp6" xmlns:xacro="http://www.ros.org/wiki/xacro">
   <property name="M_PI" value="3.14159"/>
   <link name="world">
-    <!--<inertial>
-      <mass value="0.05" />
-      <origin xyz="-0.0 0.0 -10.0" />
-      <inertia ixx="1.0" ixy="0.0" ixz="0.0"
-               iyy="1.0" iyz="0.0"
-               izz="1.0" />
-    </inertial>-->
-    <collision>
-      <origin xyz="0 0 0.15" rpy="0 0 0" />
-      <geometry>
-        <box size="0.4 0.4 0.3" />
-      </geometry>
-    </collision>
   </link>
   <joint name="base_joint" type="fixed">
@@ -27,5 +10,5 @@
 <link name="tl_base">
   <inertial>
-    <mass value="1"/>
+    <mass value="50"/>
     <inertia ixx="100" ixy="0" ixz="0" iyy="100" iyz="0" izz="100" />
     <origin xyz="0 0 0"/>
@@ -92,5 +75,5 @@
       <origin rpy="-1.57 0 0.0" xyz="0 0 0.4"/>
       <geometry>
-        <mesh filename="package://irp6_description/meshes/link1.3ds" />
+        <mesh filename="package://irp6_description/meshes/link1.stl" />
       </geometry>
     </visual>
@@ -119,5 +102,5 @@
       <origin rpy="0 0 0.0" xyz="0.455 0.0 0.0"/>
       <geometry>
-        <mesh filename="package://irp6_description/meshes/link2.3ds" />
+        <mesh filename="package://irp6_description/meshes/link2.stl" />
       </geometry>
     </visual>
@@ -145,5 +128,5 @@
       <origin rpy="0 0 1.57" xyz="0 0.67 0.0"/>
       <geometry>
-        <mesh filename="package://irp6_description/meshes/link3.3ds" />
+        <mesh filename="package://irp6_description/meshes/link3.stl" />
       </geometry>
     </visual>
@@ -151,5 +134,5 @@
       <origin rpy="0 0 1.57" xyz="0 0.67 0.0"/>
       <geometry>
-        <mesh filename="package://irp6_description/meshes/link3.stlb" scale="1.0 1.0 1.3" />
+        <mesh filename="package://irp6_description/meshes/link3b.stl" scale="1.0 1.0 1.3" />
       </geometry>
     </collision>
@@ -171,5 +154,5 @@
       <origin rpy="1.57 0 1.57" xyz="0.0 0.175 0.0"/>
       <geometry>
-        <mesh filename="package://irp6_description/meshes/link4.3ds" />
+        <mesh filename="package://irp6_description/meshes/link4.stl" />
       </geometry>
     </visual>
@@ -177,5 +160,5 @@
       <origin rpy="1.57 0 1.57" xyz="0.0 0.175 0.0"/>
       <geometry>
-        <mesh filename="package://irp6_description/meshes/link4.stlb" />
+        <mesh filename="package://irp6_description/meshes/link4b.stl" />
       </geometry>
     </collision>
@@ -197,5 +180,5 @@
       <origin rpy="1.57 0 0.0" xyz="0.0 0.0 0.19"/>
       <geometry>
-        <mesh filename="package://irp6_description/meshes/link5.3ds" />
+        <mesh filename="package://irp6_description/meshes/link5.stl" />
       </geometry>
     </visual>
@@ -203,5 +186,5 @@
       <origin rpy="1.57 0 0.0" xyz="0.0 0.0 0.19"/>
       <geometry>
-        <mesh filename="package://irp6_description/meshes/link5.stlb" />
+        <mesh filename="package://irp6_description/meshes/link5b.stl" />
       </geometry>
     </collision>
@@ -223,5 +206,5 @@
       <origin rpy="0 0 0.0" xyz="0 0.0 0.15"/>
       <geometry>
-         <mesh filename="package://irp6_description/meshes/link6.3ds" />
+         <mesh filename="package://irp6_description/meshes/link6.stl" />
       </geometry>
     </visual>
@@ -331,6 +314,6 @@
   <link name="pl_base">
     <inertial>
-      <mass value="0" />
-      <origin xyz="-0.0 0.0 0.0" />
+      <mass value="50" />
+      <origin xyz="0.0 0.0 0.0" />
       <inertia ixx="1.0" ixy="0.0" ixz="0.0"
                iyy="1.0" iyz="0.0"
@@ -369,5 +352,5 @@
       <origin rpy="-1.57 0 0.0" xyz="0 0 0.4"/>
       <geometry>
-        <mesh filename="package://irp6_description/meshes/link1.3ds" />
+        <mesh filename="package://irp6_description/meshes/link1.stl" />
       </geometry>
     </visual>
@@ -396,5 +379,5 @@
       <origin rpy="0 0 0.0" xyz="0.455 0.0 0.0"/>
       <geometry>
-        <mesh filename="package://irp6_description/meshes/link2.3ds" />
+        <mesh filename="package://irp6_description/meshes/link2.stl" />
       </geometry>
     </visual>
@@ -422,5 +405,5 @@
       <origin rpy="0 0 1.57" xyz="0 0.67 0.0"/>
       <geometry>
-        <mesh filename="package://irp6_description/meshes/link3.3ds" />
+        <mesh filename="package://irp6_description/meshes/link3.stl" />
       </geometry>
     </visual>
@@ -428,5 +411,5 @@
       <origin rpy="0 0 1.57" xyz="0 0.67 0.0"/>
       <geometry>
-        <mesh filename="package://irp6_description/meshes/link3.stlb" scale="1.0 1.0 1.3" />
+        <mesh filename="package://irp6_description/meshes/link3b.stl" scale="1.0 1.0 1.3" />
       </geometry>
     </collision>
@@ -448,5 +431,5 @@
       <origin rpy="1.57 0 1.57" xyz="0.0 0.175 0.0"/>
       <geometry>
-        <mesh filename="package://irp6_description/meshes/link4.3ds" />
+        <mesh filename="package://irp6_description/meshes/link4.stl" />
       </geometry>
     </visual>
@@ -454,5 +437,5 @@
       <origin rpy="1.57 0 1.57" xyz="0.0 0.175 0.0"/>
       <geometry>
-        <mesh filename="package://irp6_description/meshes/link4.stlb" />
+        <mesh filename="package://irp6_description/meshes/link4b.stl" />
       </geometry>
     </collision>
@@ -474,5 +457,5 @@
       <origin rpy="1.57 0 0.0" xyz="0.0 0.0 0.19"/>
       <geometry>
-        <mesh filename="package://irp6_description/meshes/link5.3ds" />
+        <mesh filename="package://irp6_description/meshes/link5.stl" />
       </geometry>
     </visual>
@@ -480,5 +463,5 @@
       <origin rpy="1.57 0 0.0" xyz="0.0 0.0 0.19"/>
       <geometry>
-        <mesh filename="package://irp6_description/meshes/link5.stlb" />
+        <mesh filename="package://irp6_description/meshes/link5b.stl" />
       </geometry>
     </collision>
@@ -500,5 +483,5 @@
       <origin rpy="0 0 0.0" xyz="0 0.0 0.15"/>
       <geometry>
-         <mesh filename="package://irp6_description/meshes/link6.3ds" />
+         <mesh filename="package://irp6_description/meshes/link6.stl" />
       </geometry>
     </visual>
@@ -554,5 +537,5 @@
       <geometry>
          <box size="0.05 0.04 0.12" />
-      </geometry>origin
+      </geometry>
     </visual>
     <collision>
@@ -577,57 +560,3 @@
 <link name="p_c_optical_frame">
 </link>
-<!-- Kinect                       -->
-<!--
-  <joint name="kinect_joint" type="fixed">
-    <origin rpy="0.0 0.87 1.58" xyz="0.715 -1.07 1.8"/>
-    <parent link="base_link"/>
-    <child link="kinect_base"/>
-  </joint>
-  <link name="kinect_base">
-  </link>
-  <joint name="kinect_depth_joint" type="fixed">
-    <origin rpy="0 0.0 0" xyz="0.0 -0.02 0.0"/>
-    <parent link="kinect_base"/>
-    <child link="openni_depth_frame"/>
-  </joint>
-  <link name="openni_depth_frame">
-  </link>
-  <joint name="kinect_rgb_joint" type="fixed">
-    <origin rpy="0 0.0 0" xyz="0.0 -0.04 0.0"/>
-    <parent link="kinect_base"/>
-    <child link="openni_rgb_frame"/>
-  </joint>
-  <link name="openni_rgb_frame">
-  </link>
-  <joint name="kinect_depth_optical_joint" type="fixed">
-    <origin xyz="0 0.0 0" rpy="1.57 0.0 1.57"/>
-    <parent link="openni_depth_frame"/>
-    <child link="openni_depth_optical_frame"/>
-  </joint>
-  <link name="openni_depth_optical_frame">
-  </link>
-  <joint name="kinect_rgb_optical_joint" type="fixed">
-    <origin xyz="0 0.0 0" rpy="1.57 0.0 1.57"/>
-    <parent link="openni_rgb_frame"/>
-    <child link="openni_rgb_optical_frame"/>
-  </joint>
-  <link name="openni_rgb_optical_frame">
-  </link>
--->
-<!--
-  <joint name="laser_tilt" type="revolute">
-    <origin rpy="${0.5 * M_PI} 0 0" xyz="0.0 -0.1 2.2"/>
-    <axis xyz="0 0 1"/>
-    <limit lower="0.0" upper="3.14" effort="10.0" velocity="10.0" />
-    <parent link="base_link"/>
-    <child link="laser_link"/>
-  </joint>
-  <link name="laser_link">
-    <inertial>
-      <mass value="0.1"/>
-      <origin xyz="0.0 0.0 0.0"/>
-      <inertia ixx="0.1" ixy="0" ixz="0" iyy="0.1" iyz="0" izz="0.1"/>
-    </inertial>
-  </link>
--->
 </robot>

Commit message: Added camera description

File: irp6_description/robots/irp6pboth.urdf.xacro (robot description, xacro)
@@ -2,4 +2,5 @@
 <robot name="irp6" xmlns:xacro="http://www.ros.org/wiki/xacro">
   <property name="M_PI" value="3.14159"/>
+  <xacro:include filename="$(find irp6_description)/robots/irp6.gazebo" />
   <link name="world">
   </link>
@@ -10,5 +11,5 @@
 <link name="tl_base">
   <inertial>
-    <mass value="50"/>
+    <mass value="100"/>
     <inertia ixx="100" ixy="0" ixz="0" iyy="100" iyz="0" izz="100" />
     <origin xyz="0 0 0"/>
@@ -32,5 +33,5 @@
 <link name="tl_t">
   <inertial>
-    <mass value="1"/>
+    <mass value="100"/>
     <inertia ixx="100" ixy="0" ixz="0" iyy="100" iyz="0" izz="100" />
     <origin xyz="0 0 0"/>
@@ -68,5 +69,5 @@
   <link name="tl_1">
     <inertial>
-      <mass value="0.1"/>
+      <mass value="50"/>
       <origin xyz="0.0 0.0 0.0"/>
       <inertia ixx="0.1" ixy="0" ixz="0" iyy="0.1" iyz="0" izz="0.1"/>
@@ -95,5 +96,5 @@
   <link name="tl_2">
     <inertial>
-      <mass value="0.1"/>
+      <mass value="20"/>
       <origin xyz="0.0 0.0 0.0"/>
       <inertia ixx="0.1" ixy="0" ixz="0" iyy="0.1" iyz="0" izz="0.1"/>
@@ -121,5 +122,5 @@
   <link name="tl_3">
     <inertial>
-      <mass value="0.1"/>
+      <mass value="20"/>
       <origin xyz="0.0 0.0 0.0"/>
       <inertia ixx="0.1" ixy="0" ixz="0" iyy="0.1" iyz="0" izz="0.1"/>
@@ -147,5 +148,5 @@
   <link name="tl_4">
     <inertial>
-      <mass value="0.1"/>
+      <mass value="15"/>
       <origin xyz="0.0 0.0 0.0"/>
       <inertia ixx="0.1" ixy="0" ixz="0" iyy="0.1" iyz="0" izz="0.1"/>
@@ -173,5 +174,5 @@
   <link name="tl_5">
     <inertial>
-      <mass value="0.1"/>
+      <mass value="15"/>
       <origin xyz="0.0 0.0 0.0"/>
       <inertia ixx="0.1" ixy="0" ixz="0" iyy="0.1" iyz="0" izz="0.1"/>
@@ -199,5 +200,5 @@
   <link name="tl_6">
     <inertial>
-      <mass value="0.1"/>
+      <mass value="5"/>
       <origin xyz="0.0 0.0 0.0"/>
       <inertia ixx="0.1" ixy="0" ixz="0" iyy="0.1" iyz="0" izz="0.1"/>
@@ -233,5 +234,5 @@
   <link name="tl_g1">
     <inertial>
-      <mass value="0.1"/>
+      <mass value="0.5"/>
       <origin xyz="0.0 0.0 0.0"/>
       <inertia ixx="0.1" ixy="0" ixz="0" iyy="0.1" iyz="0" izz="0.1"/>
@@ -252,5 +253,5 @@
 <link name="tl_g2">
     <inertial>
-      <mass value="0.1"/>
+      <mass value="0.5"/>
       <origin xyz="0.0 0.0 0.0"/>
       <inertia ixx="0.1" ixy="0" ixz="0" iyy="0.1" iyz="0" izz="0.1"/>
@@ -314,5 +315,5 @@
   <link name="pl_base">
     <inertial>
-      <mass value="50" />
+      <mass value="100" />
       <origin xyz="0.0 0.0 0.0" />
       <inertia ixx="1.0" ixy="0.0" ixz="0.0"
@@ -345,5 +346,5 @@
   <link name="pl_1">
     <inertial>
-      <mass value="0.1"/>
+      <mass value="50"/>
       <origin xyz="0.0 0.0 0.0"/>
       <inertia ixx="0.1" ixy="0" ixz="0" iyy="0.1" iyz="0" izz="0.1"/>
@@ -372,5 +373,5 @@
   <link name="pl_2">
     <inertial>
-      <mass value="0.1"/>
+      <mass value="20"/>
       <origin xyz="0.0 0.0 0.0"/>
       <inertia ixx="0.1" ixy="0" ixz="0" iyy="0.1" iyz="0" izz="0.1"/>
@@ -398,5 +399,5 @@
   <link name="pl_3">
     <inertial>
-      <mass value="0.1"/>
+      <mass value="20"/>
       <origin xyz="0.0 0.0 0.0"/>
       <inertia ixx="0.1" ixy="0" ixz="0" iyy="0.1" iyz="0" izz="0.1"/>
@@ -424,5 +425,5 @@
   <link name="pl_4">
     <inertial>
-      <mass value="0.1"/>
+      <mass value="15"/>
       <origin xyz="0.0 0.0 0.0"/>
       <inertia ixx="0.1" ixy="0" ixz="0" iyy="0.1" iyz="0" izz="0.1"/>
@@ -450,5 +451,5 @@
   <link name="pl_5">
     <inertial>
-      <mass value="0.1"/>
+      <mass value="15"/>
       <origin xyz="0.0 0.0 0.0"/>
       <inertia ixx="0.1" ixy="0" ixz="0" iyy="0.1" iyz="0" izz="0.1"/>
@@ -476,5 +477,5 @@
   <link name="pl_6">
     <inertial>
-      <mass value="0.1"/>
+      <mass value="5"/>
       <origin xyz="0.0 0.0 0.0"/>
       <inertia ixx="0.1" ixy="0" ixz="0" iyy="0.1" iyz="0" izz="0.1"/>
@@ -510,5 +511,5 @@
   <link name="pl_g1">
     <inertial>
-      <mass value="0.1"/>
+      <mass value="0.5"/>
       <origin xyz="0.0 0.0 0.0"/>
       <inertia ixx="0.1" ixy="0" ixz="0" iyy="0.1" iyz="0" izz="0.1"/>
@@ -529,5 +530,5 @@
 <link name="pl_g2">
     <inertial>
-      <mass value="0.1"/>
+      <mass value="0.5"/>
       <origin xyz="0.0 0.0 0.0"/>
       <inertia ixx="0.1" ixy="0" ixz="0" iyy="0.1" iyz="0" izz="0.1"/>

Commit message: New models format

File: irp6_description/robots/irp6pboth.urdf.xacro (robot description, xacro)
@@ -2,5 +2,5 @@
 <robot name="irp6" xmlns:xacro="http://www.ros.org/wiki/xacro">
   <property name="M_PI" value="3.14159"/>
-  <xacro:include filename="$(find irp6_description)/robots/irp6.gazebo" />
+  <xacro:include filename="$(find irp6_description)/robots/irp6both.gazebo" />
   <link name="world">
   </link>
@@ -12,5 +12,5 @@
   <inertial>
     <mass value="100"/>
-    <inertia ixx="100" ixy="0" ixz="0" iyy="100" iyz="0" izz="100" />
+    <inertia ixx="0" ixy="0" ixz="0" iyy="0" iyz="0" izz="0" />
     <origin xyz="0 0 0"/>
   </inertial>
@@ -33,6 +33,6 @@
 <link name="tl_t">
   <inertial>
-    <mass value="100"/>
-    <inertia ixx="100" ixy="0" ixz="0" iyy="100" iyz="0" izz="100" />
+    <mass value="50"/>
+    <inertia ixx="1" ixy="0" ixz="0" iyy="1" iyz="0" izz="1" />
     <origin xyz="0 0 0"/>
   </inertial>
@@ -71,10 +71,10 @@
       <mass value="50"/>
       <origin xyz="0.0 0.0 0.0"/>
-      <inertia ixx="0.1" ixy="0" ixz="0" iyy="0.1" iyz="0" izz="0.1"/>
+      <inertia ixx="10" ixy="0" ixz="0" iyy="10" iyz="0" izz="10"/>
     </inertial>
     <visual>
       <origin rpy="-1.57 0 0.0" xyz="0 0 0.4"/>
       <geometry>
-        <mesh filename="package://irp6_description/meshes/link1.stl" />
+        <mesh filename="package://irp6_description/meshes/link1.dae" />
       </geometry>
     </visual>
@@ -98,10 +98,10 @@
       <mass value="20"/>
       <origin xyz="0.0 0.0 0.0"/>
-      <inertia ixx="0.1" ixy="0" ixz="0" iyy="0.1" iyz="0" izz="0.1"/>
+      <inertia ixx="10" ixy="0" ixz="0" iyy="10" iyz="0" izz="10"/>
     </inertial>
     <visual>
       <origin rpy="0 0 0.0" xyz="0.455 0.0 0.0"/>
       <geometry>
-        <mesh filename="package://irp6_description/meshes/link2.stl" />
+        <mesh filename="package://irp6_description/meshes/link2.dae" />
       </geometry>
     </visual>
@@ -124,10 +124,10 @@
       <mass value="20"/>
       <origin xyz="0.0 0.0 0.0"/>
-      <inertia ixx="0.1" ixy="0" ixz="0" iyy="0.1" iyz="0" izz="0.1"/>
+      <inertia ixx="10" ixy="0" ixz="0" iyy="10" iyz="0" izz="10"/>
     </inertial>
     <visual>
       <origin rpy="0 0 1.57" xyz="0 0.67 0.0"/>
       <geometry>
-        <mesh filename="package://irp6_description/meshes/link3.stl" />
+        <mesh filename="package://irp6_description/meshes/link3.dae" />
       </geometry>
     </visual>
@@ -135,5 +135,5 @@
       <origin rpy="0 0 1.57" xyz="0 0.67 0.0"/>
       <geometry>
-        <mesh filename="package://irp6_description/meshes/link3b.stl" scale="1.0 1.0 1.3" />
+        <mesh filename="package://irp6_description/meshes/link3b.dae" scale="1.0 1.0 1.3" />
       </geometry>
     </collision>
@@ -150,10 +150,10 @@
       <mass value="15"/>
       <origin xyz="0.0 0.0 0.0"/>
-      <inertia ixx="0.1" ixy="0" ixz="0" iyy="0.1" iyz="0" izz="0.1"/>
+      <inertia ixx="10" ixy="0" ixz="0" iyy="10" iyz="0" izz="10"/>
     </inertial>
     <visual>
       <origin rpy="1.57 0 1.57" xyz="0.0 0.175 0.0"/>
       <geometry>
-        <mesh filename="package://irp6_description/meshes/link4.stl" />
+        <mesh filename="package://irp6_description/meshes/link4.dae" />
       </geometry>
     </visual>
@@ -161,5 +161,5 @@
       <origin rpy="1.57 0 1.57" xyz="0.0 0.175 0.0"/>
       <geometry>
-        <mesh filename="package://irp6_description/meshes/link4b.stl" />
+        <mesh filename="package://irp6_description/meshes/link4b.dae" />
       </geometry>
     </collision>
@@ -176,10 +176,10 @@
       <mass value="15"/>
       <origin xyz="0.0 0.0 0.0"/>
-      <inertia ixx="0.1" ixy="0" ixz="0" iyy="0.1" iyz="0" izz="0.1"/>
+      <inertia ixx="10" ixy="0" ixz="0" iyy="10" iyz="0" izz="10"/>
     </inertial>
     <visual>
       <origin rpy="1.57 0 0.0" xyz="0.0 0.0 0.19"/>
       <geometry>
-        <mesh filename="package://irp6_description/meshes/link5.stl" />
+        <mesh filename="package://irp6_description/meshes/link5.dae" />
       </geometry>
     </visual>
@@ -187,5 +187,5 @@
       <origin rpy="1.57 0 0.0" xyz="0.0 0.0 0.19"/>
       <geometry>
-        <mesh filename="package://irp6_description/meshes/link5b.stl" />
+        <mesh filename="package://irp6_description/meshes/link5b.dae" />
       </geometry>
     </collision>
@@ -202,10 +202,10 @@
       <mass value="5"/>
       <origin xyz="0.0 0.0 0.0"/>
-      <inertia ixx="0.1" ixy="0" ixz="0" iyy="0.1" iyz="0" izz="0.1"/>
+      <inertia ixx="10" ixy="0" ixz="0" iyy="10" iyz="0" izz="10"/>
     </inertial>
     <visual>
       <origin rpy="0 0 0.0" xyz="0 0.0 0.15"/>
       <geometry>
-         <mesh filename="package://irp6_description/meshes/link6.stl" />
+         <mesh filename="package://irp6_description/meshes/link6.dae" />
       </geometry>
     </visual>
@@ -236,5 +236,5 @@
       <mass value="0.5"/>
       <origin xyz="0.0 0.0 0.0"/>
-      <inertia ixx="0.1" ixy="0" ixz="0" iyy="0.1" iyz="0" izz="0.1"/>
+      <inertia ixx="10" ixy="0" ixz="0" iyy="10" iyz="0" izz="10"/>
     </inertial>
     <visual>
@@ -255,5 +255,5 @@
       <mass value="0.5"/>
       <origin xyz="0.0 0.0 0.0"/>
-      <inertia ixx="0.1" ixy="0" ixz="0" iyy="0.1" iyz="0" izz="0.1"/>
+      <inertia ixx="10" ixy="0" ixz="0" iyy="10" iyz="0" izz="10"/>
     </inertial>
     <visual>
@@ -348,10 +348,10 @@
       <mass value="50"/>
       <origin xyz="0.0 0.0 0.0"/>
-      <inertia ixx="0.1" ixy="0" ixz="0" iyy="0.1" iyz="0" izz="0.1"/>
+      <inertia ixx="10" ixy="0" ixz="0" iyy="10" iyz="0" izz="10"/>
     </inertial>
     <visual>
       <origin rpy="-1.57 0 0.0" xyz="0 0 0.4"/>
       <geometry>
-        <mesh filename="package://irp6_description/meshes/link1.stl" />
+        <mesh filename="package://irp6_description/meshes/link1.dae" />
       </geometry>
     </visual>
@@ -375,10 +375,10 @@
       <mass value="20"/>
       <origin xyz="0.0 0.0 0.0"/>
-      <inertia ixx="0.1" ixy="0" ixz="0" iyy="0.1" iyz="0" izz="0.1"/>
+      <inertia ixx="10" ixy="0" ixz="0" iyy="10" iyz="0" izz="10"/>
     </inertial>
     <visual>
       <origin rpy="0 0 0.0" xyz="0.455 0.0 0.0"/>
       <geometry>
-        <mesh filename="package://irp6_description/meshes/link2.stl" />
+        <mesh filename="package://irp6_description/meshes/link2.dae" />
       </geometry>
     </visual>
@@ -401,10 +401,10 @@
       <mass value="20"/>
       <origin xyz="0.0 0.0 0.0"/>
-      <inertia ixx="0.1" ixy="0" ixz="0" iyy="0.1" iyz="0" izz="0.1"/>
+      <inertia ixx="10" ixy="0" ixz="0" iyy="10" iyz="0" izz="10"/>
     </inertial>
     <visual>
       <origin rpy="0 0 1.57" xyz="0 0.67 0.0"/>
       <geometry>
-        <mesh filename="package://irp6_description/meshes/link3.stl" />
+        <mesh filename="package://irp6_description/meshes/link3.dae" />
       </geometry>
     </visual>
@@ -412,5 +412,5 @@
       <origin rpy="0 0 1.57" xyz="0 0.67 0.0"/>
       <geometry>
-        <mesh filename="package://irp6_description/meshes/link3b.stl" scale="1.0 1.0 1.3" />
+        <mesh filename="package://irp6_description/meshes/link3b.dae" scale="1.0 1.0 1.3" />
       </geometry>
     </collision>
@@ -427,10 +427,10 @@
       <mass value="15"/>
       <origin xyz="0.0 0.0 0.0"/>
-      <inertia ixx="0.1" ixy="0" ixz="0" iyy="0.1" iyz="0" izz="0.1"/>
+      <inertia ixx="10" ixy="0" ixz="0" iyy="10" iyz="0" izz="10"/>
     </inertial>
     <visual>
       <origin rpy="1.57 0 1.57" xyz="0.0 0.175 0.0"/>
       <geometry>
-        <mesh filename="package://irp6_description/meshes/link4.stl" />
+        <mesh filename="package://irp6_description/meshes/link4.dae" />
       </geometry>
     </visual>
@@ -438,5 +438,5 @@
       <origin rpy="1.57 0 1.57" xyz="0.0 0.175 0.0"/>
       <geometry>
-        <mesh filename="package://irp6_description/meshes/link4b.stl" />
+        <mesh filename="package://irp6_description/meshes/link4b.dae" />
       </geometry>
     </collision>
@@ -453,10 +453,10 @@
       <mass value="15"/>
       <origin xyz="0.0 0.0 0.0"/>
-      <inertia ixx="0.1" ixy="0" ixz="0" iyy="0.1" iyz="0" izz="0.1"/>
+      <inertia ixx="10" ixy="0" ixz="0" iyy="10" iyz="0" izz="10"/>
     </inertial>
     <visual>
       <origin rpy="1.57 0 0.0" xyz="0.0 0.0 0.19"/>
       <geometry>
-        <mesh filename="package://irp6_description/meshes/link5.stl" />
+        <mesh filename="package://irp6_description/meshes/link5.dae" />
       </geometry>
     </visual>
@@ -464,5 +464,5 @@
       <origin rpy="1.57 0 0.0" xyz="0.0 0.0 0.19"/>
       <geometry>
-        <mesh filename="package://irp6_description/meshes/link5b.stl" />
+        <mesh filename="package://irp6_description/meshes/link5b.dae" />
       </geometry>
     </collision>
@@ -479,10 +479,10 @@
       <mass value="5"/>
       <origin xyz="0.0 0.0 0.0"/>
-      <inertia ixx="0.1" ixy="0" ixz="0" iyy="0.1" iyz="0" izz="0.1"/>
+      <inertia ixx="10" ixy="0" ixz="0" iyy="10" iyz="0" izz="10"/>
     </inertial>
     <visual>
       <origin rpy="0 0 0.0" xyz="0 0.0 0.15"/>
       <geometry>
-         <mesh filename="package://irp6_description/meshes/link6.stl" />
+         <mesh filename="package://irp6_description/meshes/link6.dae" />
       </geometry>
     </visual>
@@ -513,5 +513,5 @@
       <mass value="0.5"/>
       <origin xyz="0.0 0.0 0.0"/>
-      <inertia ixx="0.1" ixy="0" ixz="0" iyy="0.1" iyz="0" izz="0.1"/>
+      <inertia ixx="10" ixy="0" ixz="0" iyy="10" iyz="0" izz="10"/>
     </inertial>
     <visual>
@@ -532,5 +532,5 @@
       <mass value="0.5"/>
       <origin xyz="0.0 0.0 0.0"/>
-      <inertia ixx="0.1" ixy="0" ixz="0" iyy="0.1" iyz="0" izz="0.1"/>
+      <inertia ixx="10" ixy="0" ixz="0" iyy="10" iyz="0" izz="10"/>
     </inertial>
     <visual>
